File: Pinout.kicad_sch (KiCad schematic)
At the start: 16 parts, among them J1 Conn_01x10_Male, J10 Conn_01x12_Male, J11 Conn_01x12_Male, J12 Conn_01x08_Male, J13 Conn_01x03_Male, J14 Conn_01x02_Female, J15 Conn_01x04_Male, J2 Conn_01x13_Male, J3 Conn_01x12_Male, J4 Conn_01x13_Male, J5 Conn_01x13_Male, J6 Conn_01x04_Male, J7 Conn_01x03_Male, J8 Conn_01x17_Male, J9 Conn_01x16_Male

Commit message: Final
Parts:
- removed J8: Conn_01x17_Male, Connector_PinHeader_2.54mm:PinHeader_1x17_P2.54mm_Vertical, symbol Connector:Conn_01x17_Male
- removed J9: Conn_01x16_Male, Connector_PinHeader_2.54mm:PinHeader_1x16_P2.54mm_Vertical, symbol Connector:Conn_01x16_Male
- added J10, J12: Conn_01x10_Male, Connector_PinHeader_2.54mm:PinHeader_1x10_P2.54mm_Vertical, symbol Connector:Conn_01x10_Male
- added J11, J9: Conn_01x06_Male, Connector_PinHeader_2.54mm:PinHeader_1x06_P2.54mm_Vertical, symbol Connector:Conn_01x06_Male
- added J8: Conn_01x01_Male, Connector_PinHeader_2.54mm:PinHeader_1x01_P2.54mm_Vertical, symbol Connector:Conn_01x01_Male
- renumbered J10 to J13, J11 to J14, J12 to J15, J13 to J16, J14 to J17, J15 to J18
Connections:
- net CAM0_C_N: now also J9.1 (Pin_1)
- net CAM0_C_P: now also J9.2 (Pin_2)
- net CAM0_D0_N: now also J9.3 (Pin_3)
- net CAM0_D0_P: now also J9.4 (Pin_4)
- net CAM0_D1_N: now also J9.5 (Pin_5)
- net CAM0_D1_P: now also J9.6 (Pin_6)
- net CAM1_C_N: now also J10.1 (Pin_1)
- net CAM1_C_P: now also J10.2 (Pin_2)
- net CAM1_D0_N: now also J10.3 (Pin_3)
- net CAM1_D0_P: now also J10.4 (Pin_4)
- net CAM1_D1_N: now also J10.5 (Pin_5)
- net CAM1_D1_P: now also J10.6 (Pin_6)
- net CAM1_D2_N: now also J10.7 (Pin_7)
- net CAM1_D2_P: now also J10.8 (Pin_8)
- net CAM1_D3_N: now also J10.9 (Pin_9)
- net CAM1_D3_P: now also J10.10 (Pin_10)
- net DSI0_C_N: now also J11.1 (Pin_1)
- net DSI0_C_P: now also J11.2 (Pin_2)
- net DSI0_D0_N: now also J11.3 (Pin_3)
- net DSI0_D0_P: now also J11.4 (Pin_4)
- net DSI0_D1_N: now also J11.5 (Pin_5)
- net DSI0_D1_P: now also J11.6 (Pin_6)
- net DSI1_C_N: now also J12.1 (Pin_1)
- net DSI1_C_P: now also J12.2 (Pin_2)
- net DSI1_D0_N: now also J12.3 (Pin_3)
- net DSI1_D0_P: now also J12.4 (Pin_4)
- net DSI1_D1_N: now also J12.5 (Pin_5)
- net DSI1_D1_P: now also J12.6 (Pin_6)
- net DSI1_D2_N: now also J12.7 (Pin_7)
- net DSI1_D2_P: now also J12.8 (Pin_8)
- net DSI1_D3_N: now also J12.9 (Pin_9)
- net DSI1_D3_P: now also J12.10 (Pin_10)
- net VDAC_COMP: now also J8.1 (Pin_1)
Other:
- moved on the sheet: J13, J14, J16
